File: pcb/internal-sdcard-interface/internal-sdcard-interface.kicad_sch (KiCad schematic)
At the start: 77 parts, among them J1 EXPANSION BOARD, J2 POWER, J3 TERMINAL, J5 SDCARD, U1 74HC04, U10 74HC173, U11 74HC245, U12 74HC157, U17 74HC85, U18 74HC00, U19 74HC00, U2 CY62256-70PC, U20 74HC02, U21 74HC123, U23 74HC163, U24 74HC138, U25 74HC138, U26 74HC32, U27 74HC00, U29 74HC165, U3 74HC00, U30 74HC595, U31 74HC273, U32 74HC273, U33 SST39SF010, U34 CY62128ELL-45SXI, U4 CY62256-70PC, U5 74HC74, U6 74HC74, U7 74HC32, U8 74HC688, U9 74HC32, X1 16MHz

Commit message: Updating session
Parts:
- J1: footprint Connector_PinHeader_2.54mm:PinHeader_2x20_P2.54mm_Vertical -> Connector_IDC:IDC-Header_2x20_P2.54mm_Vertical
- J2: symbol Connector:Conn_01x02_Male -> Connector:Conn_01x02_Pin
Other:
- note added: "A cheap pre-made SD-CARD interface board is used. This board does the voltage translation (3.3 <-> 5V) via an op amp. (DEBO MICROSD2 on Reichelt)"
- note added: "ADDRESS REGISTERS"
- note added: "I/O PORT MULTIPLEXER"
- note added: "PINOUT: see also Field Support Manual: Diagram 3.8.1"
- note added: "RAM BANK CIRCUITRY"
- note added: "RAM BANKING REGISTER"
- note added: "Reading from 0x94 allows to extract current banking value."
- note added: "SD-CARD DAUGHTER BOARD"
- note added: "This components gives the clock signal to drive the SPI protocol. Although it was designed around a 16 MHz osscillator, benchmarks indicate that any frequency between 4 - 16.25 MHz works fine."
- note added: "Via a ribbon cable, this 40 pin interface port is connected to the main board of the P2000T."
- note removed: "BANK SWITCHING LOGICS"
- note removed: "SELECTION COMPONENT"
- note removed: "See also Field Support Manual: Diagram 3.8.1"
- moved on the sheet: C1, C10, C11, C12, C18, C19, C2, C20, C21, C22, C23, C24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
