File: pcb/port2-sdcard-gen2/port2-sdcard-gen2.kicad_sch (KiCad schematic)
At the start: 13 parts, among them J1 Micro_SD_Card_Det1, J2 P2000T Port 2, U1 CY62128ELL-45SXI, U12 74HC165, U13 74HC595, U15 SST39SF010, U16 AMS1117-3.3, U21 74LVC125

Commit message: Initial prototype schematic
Parts:
- added D1, D2, D3, D4, D5, D6, D7, D8: 1N4148, Diode_THT:D_DO-35_SOD27_P7.62mm_Horizontal, symbol Device:D
- added D10: WRITE, LED_THT:LED_D5.0mm, symbol Device:LED
- added D9: READ, LED_THT:LED_D5.0mm, symbol Device:LED
- added J1: Atmel-JTAG-10, Connector_IDC:IDC-Header_2x05_P2.54mm_Vertical, symbol atf1504_plcc44_breakout:Atmel-JTAG-10
- added J2: PLAYER1, Connector_Dsub:DSUB-9_Male_Horizontal_P2.77x2.84mm_EdgePinOffset4.94mm_Housed_MountingHolesOffset7.48mm, symbol atari:joystick
- added J3: POWER, symbol Connector:Conn_01x02_Pin
- added J4: PLAYER2, Connector_Dsub:DSUB-9_Male_Horizontal_P2.77x2.84mm_EdgePinOffset4.94mm_Housed_MountingHolesOffset7.48mm, symbol atari:joystick
- added R1: 10k, symbol Device:R
- added R2, R3: 1k, Resistor_THT:R_Axial_DIN0207_L6.3mm_D2.5mm_P7.62mm_Horizontal, symbol Device:R
- added R8: 180, Resistor_SMD:R_0805_2012Metric_Pad1.20x1.40mm_HandSolder, symbol Device:R
- added R9: 560, Resistor_SMD:R_0805_2012Metric_Pad1.20x1.40mm_HandSolder, symbol Device:R
- added RN1: 1k, Resistor_THT:R_Array_SIP9, symbol Device:R_Network08_US
- added U1: ~, symbol ATF1504AS-10AU100:ATF1504AS-10AU100
- added U4: 74HC74, Package_SO:SO-14_3.9x8.65mm_P1.27mm, symbol 74xx:74HC74
- added U5: 74HC00, Package_SO:SO-14_3.9x8.65mm_P1.27mm, symbol 74xx:74HC00
- added unit 5 of U6
- added X1: 16MHz, Oscillator:Oscillator_DIP-14, symbol Oscillator:TCXO-14
- renumbered C23 to C1, J2 to J5, J1 to J6, R9 to R4, R11 to R5, R10 to R6, R8 to R7, U15 to U2, U1 to U3, U21 to U6, U16 to U7, U12 to U8, U13 to U9
Connections:
- net +3V3: now also U6.14 (VCC)
- net A0: now also U1.29 (I/O)
- net A1: now also U1.30 (I/O)
- net A2: now also U1.31 (I/O)
- net A3: now also U1.32 (I/O)
- net A4: now also U1.33 (I/O)
- net A5: now also U1.35 (I/O)
- net A6: now also U1.36 (I/O)
- net A7: now also U1.37 (I/O)
- net CA0: now also U1.52 (I/O)
- net CA1: now also U1.54 (I/O)
- net CA10: now also U1.67 (I/O)
- net CA11: now also U1.68 (I/O)
- net CA12: now also U1.69 (I/O)
- net CA13: now also U1.71 (I/O)
- net CA14: now also U1.75 (I/O)
- net CA15: now also U1.76 (I/O)
- net CA2: now also U1.56 (I/O)
- net CA3: now also U1.57 (I/O)
- net CA4: now also U1.58 (I/O)
- net CA5: now also U1.60 (I/O)
- net CA6: now also U1.61 (I/O)
- net CA7: now also U1.63 (I/O)
- net CA8: now also U1.64 (I/O)
- net CA9: now also U1.65 (I/O)
- net CLK: now also U1.16 (I/O), U5.1, U5.2
- net D0: now also D1.2 (A), U1.40 (I/O), U4.2 (D)
- net D1: now also D2.2 (A), U1.41 (I/O), U4.12 (D)
- net D2: now also D3.2 (A), U1.42 (I/O/PD2)
- net D3: now also D4.2 (A), U1.44 (I/O)
- net D4: now also D5.2 (A), U1.45 (I/O)
- net D5: now also D6.2 (A), U1.46 (I/O)
- net D6: now also D7.2 (A), U1.47 (I/O)
- net D7: now also D8.2 (A), U1.48 (I/O)
- net GND: now also D10.1 (K), D9.1 (K), J1.10 (GND), J1.2 (GND), J2.8 (CC-DPAD), J2.9 (CC-FIRE), J3.2 (Pin_2), J4.8 (CC-DPAD), J4.9 (CC-FIRE), U1.11 (GND), U1.26 (GND), U1.38 (GND), U1.43 (GND), U1.59 (GND), U1.74 (GND), U1.86 (GND), U1.95 (GND), U4.7 (GND), U5.12, U5.13, U5.7 (GND), U6.7 (GND), X1.7 (GND)
- net MISO: now also R1.1
- net RAM16: now also U1.80 (I/O)
- net ROM16: now also U1.79 (I/O)
- net VCC: now also J1.4 (VccT), J2.5 (VCC), J3.1 (Pin_1), J4.5 (VCC), R2.1, R3.1, RN1.1 (common), U1.18 (VCCIO), U1.3 (VCCIO), U1.34 (VCCIO), U1.39 (VCCINT), U1.51 (VCCIO), U1.66 (VCCIO), U1.82 (VCCIO), U1.91 (VCCINT), U4.10 (~{S}), U4.14 (VCC), U4.4 (~{S}), U5.14 (VCC), X1.14 (Vcc)
- net ~{CLK}: now also U5.3
- net ~{CS}: now also U1.94 (I/O)
- net ~{IORQ}: now also U1.21 (I/O)
- net ~{RD}: now also U1.88 (INPUT/OE1)
- net ~{RES}: now also U1.89 (INPUT/GCLR), U4.1 (~{R}), U4.13 (~{R})
- net ~{SER_RD}: now also U1.19 (I/O)
- net ~{SER_WR}: now also U1.20 (I/O)
- net ~{WR}: now also U1.90 (INPUT/OE2/GCLK2)
- net ~{S13} renamed ~{ROMCS}
- net ~{ROMCS}: now also U1.81 (I/O)
- net ~{S14} renamed ~{RAMCS}
- net ~{RAMCS}: now also U1.83 (I/O)
- new net: R1.2, U1.8 (I/O)
- new net: R8.1, U4.5 (Q)
- new net: D9.2 (A), R8.2
- new net: D10.2 (A), R9.2
- new net: R9.1, U4.9 (Q)
- new net 16MHz: U1.87 (INPUT/GCLK1), X1.8 (OUT)
- new net JD0: D1.1 (K), U1.84 (I/O)
- new net JD1: D2.1 (K), U1.85 (I/O/GCLK3)
- new net JD2: D3.1 (K), U1.23 (I/O)
- new net JD3: D4.1 (K), U1.25 (I/O)
- new net JD4: D5.1 (K), U1.92 (I/O)
- new net JD5: D6.1 (K), U1.93 (I/O)
- new net JD6: D7.1 (K), U1.6 (I/O)
- new net JD7: D8.1 (K), J1.3 (TDO), U1.73 (I/O/TDO)
- new net LED_SEL: U1.17 (I/O), U4.11 (C), U4.3 (C)
- new net TCK: J1.1 (TCK), U1.62 (I/O/TCK)
- new net TDI: J1.9 (TDI), U1.4 (I/O/TDI)
- new net TMS: J1.5 (TMS), U1.15 (I/O/TMS)
- new net ~{P1_DOWN}: J2.2 (DOWN), RN1.3 (R2), U1.99 (I/O)
- new net ~{P1_FIRE}: J2.6 (FIRE), RN1.6 (R5), U1.96 (I/O)
- new net ~{P1_LEFT}: J2.3 (LEFT), RN1.4 (R3), U1.98 (I/O)
- new net ~{P1_RIGHT}: J2.4 (RIGHT), RN1.5 (R4), U1.97 (I/O)
- new net ~{P1_UP}: J2.1 (UP), RN1.2 (R1), U1.100 (I/O)
- new net ~{P2_DOWN}: J4.2 (DOWN), RN1.8 (R7), U1.13 (I/O)
- new net ~{P2_FIRE}: J4.6 (FIRE), R3.2, U1.9 (I/O)
- new net ~{P2_LEFT}: J4.3 (LEFT), RN1.9 (R8), U1.12 (I/O/PD1)
- new net ~{P2_RIGHT}: J4.4 (RIGHT), R2.2, U1.10 (I/O)
- new net ~{P2_UP}: J4.1 (UP), RN1.7 (R6), U1.14 (I/O)
- no-connect marks 12 -> 17
Other:
- note added: "Atari 2600-style joysticks have one d-pad and one fire button. Atari 7800-style joysticks are partly compatible with this interface, though the secondary fire button will *not* work."
- note added: "Atari joystick pinout requires all pins to be pulled high via a resistor. Upon connect, they are brought low."
- note added: "Note: 74LVC125 needs 3v3 on VCC"
- note added: "Serial CLK"
- note added: "Set pull-up/down for MISO"
- note added: "TDO / JD7 share same pin!"
- moved on the sheet: C1, J5, J6, R4, R5, R6, R7, U2, U3, U6A, U6B, U6C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

Commit message: Initial placement components
Parts:
- D10, D9: footprint LED_THT:LED_D5.0mm -> LED_SMD:LED_0805_2012Metric_Pad1.15x1.40mm_HandSolder
- J2, J4: footprint Connector_Dsub:DSUB-9_Male_Horizontal_P2.77x2.84mm_EdgePinOffset4.94mm_Housed_MountingHolesOffset7.48mm -> Connector_Dsub:DSUB-9_Pins_Horizontal_P2.77x2.84mm_EdgePinOffset4.94mm_Housed_MountingHolesOffset4.94mm
- R1: footprint (none) -> Resistor_SMD:R_0805_2012Metric_Pad1.20x1.40mm_HandSolder
- U1: footprint (none) -> Package_QFP:TQFP-100_14x14mm_P0.5mm
- U3: footprint Package_SO:SSOP-32_11.305x20.495mm_P1.27mm -> Package_SO:SOP-32_11.305x20.495mm_P1.27mm
Changed lines of the file:
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@@
 			)
 		)
-		(property "Footprint" ""
+		(property "Footprint" "Resistor_SMD:R_0805_2012Metric_Pad1.20x1.40mm_HandSolder"
 			(at 26.67 69.088 90)
 			(effects
@@
 			)
 		)
-		(property "Footprint" "Connector_Dsub:DSUB-9_Male_Horizontal_P2.77x2.84mm_EdgePinOffset4.94mm_Housed_MountingHolesOffset7.48mm"
+		(property "Footprint" "Connector_Dsub:DSUB-9_Pins_Horizontal_P2.77x2.84mm_EdgePinOffset4.94mm_Housed_MountingHolesOffset4.94mm"
 			(at 101.6 204.47 0)
 			(effects
@@
 			)
 		)
-		(property "Footprint" "Connector_Dsub:DSUB-9_Male_Horizontal_P2.77x2.84mm_EdgePinOffset4.94mm_Housed_MountingHolesOffset7.48mm"
+		(property "Footprint" "Connector_Dsub:DSUB-9_Pins_Horizontal_P2.77x2.84mm_EdgePinOffset4.94mm_Housed_MountingHolesOffset4.94mm"
 			(at 62.23 204.47 0)
 			(effects
@@
 			)
 		)
-		(property "Footprint" "LED_THT:LED_D5.0mm"
+		(property "Footprint" "LED_SMD:LED_0805_2012Metric_Pad1.15x1.40mm_HandSolder"
 			(at 382.27 62.23 0)
 			(effects
@@
 			)
 		)
-		(property "Footprint" "LED_THT:LED_D5.0mm"
+		(property "Footprint" "LED_SMD:LED_0805_2012Metric_Pad1.15x1.40mm_HandSolder"
 			(at 382.143 52.705 0)
 			(effects
@@
 			)
 		)
-		(property "Footprint" "Package_SO:SSOP-32_11.305x20.495mm_P1.27mm"
+		(property "Footprint" "Package_SO:SOP-32_11.305x20.495mm_P1.27mm"
 			(at 246.38 74.93 0)
 			(effects
@@
 			)
 		)
-		(property "Footprint" ""
+		(property "Footprint" "Package_QFP:TQFP-100_14x14mm_P0.5mm"
 			(at 78.74 81.28 0)
 			(effects
